File: Tuan Circuit Design LM5155/PCB Design LM5155 Boost Converter.kicad_sch (KiCad schematic)
At the start: 35 parts, among them Q1 BSC035N04LS G, U1 LM5155_DSSR

Commit message: Add resistor
Parts:
- added R9: 0, Resistor_SMD:R_0402_1005Metric_Pad0.72x0.64mm_HandSolder, symbol Device:R
Connections:
- net GND: now also R9.1
- net GNDPWR: now also R9.2

Commit message: Add switch
Parts:
- added Q2: BSC035N04LS G, INF-PG-TDSON-8:INF-PG-TDSON-8, symbol BSC035N04LS G:BSC035N04LS G
- added S1: 100SP1T1B4M2QE, SW_100SP1T1B4M2QE:SW_100SP1T1B4M2QE, symbol 100SP1T1B4M2QE:100SP1T1B4M2QE
Connections:
- net INDUCTOR: now also Q2.1 (SOURCE), Q2.2 (SOURCE), Q2.3 (SOURCE); no longer Vin1.2
- new net: Q2.4 (GATE), S1.3
- new net: Q2.5 (DRAIN), Q2.6 (DRAIN), Q2.7 (DRAIN), Q2.8 (DRAIN), S1.2, Vin1.2
- no-connect marks 1 -> 2

Commit message: Update voltage protection (TVS and Fuse)
Parts:
- added D5: D_TVS, Diode_SMD:D_SMB_Handsoldering, symbol Device:D_TVS
- added F1: Fuse, Fuse:Fuse_1206_3216Metric_Pad1.42x1.75mm_HandSolder, symbol Device:Fuse
Connections:
- net COUT: now also F1.1; no longer C7.1, C8.1, C9.1, RLED1.2, Vout1.1
- net GNDPWR: now also D5.1 (A1)
- new net: C7.1, C8.1, C9.1, D5.2 (A2), F1.2, RLED1.2, Vout1.1
