File: Tuan Circuit Design LM5155/PCB Design LM5155 Boost Converter.kicad_pcb (KiCad board)
At the start: 4 copper layers, 80 x 53 mm, 45 parts, among them Q1 BSC035N04LS G, Q2 BSC035N04LS G, U1 LM5155_DSSR

Commit message: Update silkscreen
Parts:
- removed the REF** at (187.8, 92.2)
- removed the REF** at (120.3, 52.2)
- removed the REF** at (187.3, 52.2)
- added REF**: MountingHole_5mm, MountingHole:MountingHole_5mm, F.Cu at (182.3, 52.2)
- added REF**: MountingHole_5mm, MountingHole:MountingHole_5mm, F.Cu at (182.8, 92.2)
- added REF**: MountingHole_5mm, MountingHole:MountingHole_5mm, F.Cu at (115.3, 52.2)
- moved C1 5.00 mm to (140.3, 80.8)
- moved C10 5.00 mm to (160.6, 79.6)
- moved C11 5.00 mm to (162.5, 72.5)
- moved C12 5.00 mm to (160.6, 73.3)
- moved C13 5.00 mm to (164.4, 79.6)
- moved C14 5.00 mm to (170.7, 61.5)
- moved C15 5.00 mm to (171.4, 74.5)
- moved C16 5.00 mm to (168.2, 77.9)
- moved C17 5.00 mm to (166.3, 77.9)
- moved C2 5.00 mm to (140.3, 73.2)
- moved C3 5.00 mm to (131.8, 75.1)
- moved C4 5.00 mm to (132.9, 64.6)
- moved C5 5.00 mm to (153.4, 87.2)
- moved C6 5.00 mm to (150.5, 79.0)
- moved C7 5.00 mm to (146.6, 93.9)
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Other:
- board text added: "(+18V ) (4.5 A Max)"
- board text added: "3s, 4s Lipo Battery"
- board text added: "Made by Tuan Quang and Chad Copyright: UCIF1tenth(Auto Zots)"
- board text added: "Power system board version 2.0 Supply 3s and 4s lipo battery"
