File: Power System PCB For Lidar and Jetson Orin Nano/PCB Design LM5155 Boost Converter.kicad_pcb (KiCad board)
At the start: 4 copper layers, 80 x 53 mm, 79 parts, among them J1 Conn_01x04_Pin, J2 B5B-XH-A, J5 BM06B-SRSS-TBLFSN, J6 B4B-XH-A, Q1 BSC035N04LS G, Q2 BSC035N04LS G, U1 LM5155_DSSR, U2 TPS552892RYQR

Commit message: Adjust some wire
Parts:
- R6: value 360k -> 340k
- renumbered J5 to +12V, Vout4 to +18V, Vout3 to +18V
Routing:
- net /VIN: track 71.1 -> 42.7 mm
- net Net-(U2-FB): track 7.54 -> 8.48 mm
