File: Power System PCB For Lidar and Jetson Orin Nano/PCB Design LM5155 Boost Converter.kicad_pcb (KiCad board)
At the start: 4 copper layers, 80 x 53 mm, 79 parts, among them J1 Conn_01x04_Pin, J2 B5B-XH-A, J6 B4B-XH-A, Q1 BSC035N04LS G, Q2 BSC035N04LS G, U1 LM5155_DSSR, U2 TPS552892RYQR

Commit message: Update Silkscreen Backboard
Other:
- board text added: "Last Update: May 20 2026"
- board text added: "https://github.com/uci-f1tenth/Power-board.git"
Changed lines of the file:
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@@
+		)
+	)
+	(gr_text "https://github.com/uci-f1tenth/Power-board.git"
+		(at 180.5 65.5 0)
+		(layer "B.SilkS")
+		(effects
+			(font
+				(size 1.5 1.5)
+				(thickness 0.3)
+				(bold yes)
+			)
+			(justify left bottom mirror)
+		)
+	)
+	(gr_text "Last Update: May 20 2026"
+		(at 180.5 68.5 0)
+		(layer "B.SilkS")
+		(effects
+			(font
+				(size 1.5 1.5)
+				(thickness 0.3)
+				(bold yes)
+			)
+			(justify left bottom mirror)
 		)
 	)

Commit message: Update
Parts:
- renumbered +12V to J5, +18V to Vout3, +18V to Vout4
Changed lines of the file:
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@@
 		(layer "F.Cu")
 		(at 145.1 98.811 180)
-		(property "Reference" "+18V"
+		(property "Reference" "Vout4"
 			(at -2.4 -4.289 0)
 			(layer "F.SilkS")
@@
 		(layer "F.Cu")
 		(at 138.115 98.811 180)
-		(property "Reference" "+18V"
+		(property "Reference" "Vout3"
 			(at -1.885 -4.189 0)
 			(layer "F.SilkS")
@@
 		(at 127.955 92.461)
 		(tags "BM06B-SRSS-TBLFSN ")
-		(property "Reference" "+12V"
+		(property "Reference" "J5"
 			(at 6.545 -0.261 0)
 			(unlocked yes)
