File: Power System PCB For Lidar and Jetson Orin Nano/PCB Design LM5155 Boost Converter.kicad_pcb (KiCad board)
At the start: 4 copper layers, 80 x 53 mm, 79 parts, among them J1 Conn_01x04_Pin, J2 B5B-XH-A, J6 B4B-XH-A, Q1 BSC035N04LS G, Q2 BSC035N04LS G, U1 LM5155_DSSR, U2 TPS552892RYQR

Commit message: Adjust some stuff
Parts:
- added Vin: TB002-500-02BE, 282834-2:TE_282834-2, F.Cu at (183.5, 88.3)
- moved Vout 4.20 mm to (183.8, 80.6)
- moved D7 4.09 mm to (132.7, 87.0)
- moved S1 1.66 mm to (183.8, 73.0)
- moved R19 1.38 mm to (128.9, 86.9), turned to 0 degrees
- moved Q2 1.02 mm to (181.9, 66.0)
- moved R20 0.64 mm to (128.9, 85.7), turned to 0 degrees
- moved J5 0.40 mm to (128.3, 92.7)
- renumbered +18V to +12V, +12V to J5, Vout5 to Vout
Connections:
- +12V pad 1: Net-(D5-A2) -> /Vout2
Routing:
- net /Vout2: track 20.1 -> 43.2 mm
- net Net-(D5-A2): track 31.0 -> 22.3 mm
- net GNDPWR: track 94.0 -> 86.1 mm, vias 23 -> 20
- net /INDUCTOR: track 28.2 -> 26.5 mm
- net /VIN: track 42.7 -> 44.1 mm
- net Net-(Q2-GATE): track 5.67 -> 5.09 mm
Other:
- board text added: "Servo"
